Commit message: Removed battery and added imu to the robot

File: src/scooter_simulator/ackermann_vehicle-noetic/ackermann_vehicle_description/urdf/em_3905.urdf.xacro (robot description, xacro)
@@ -41,5 +41,5 @@
        battery_length is measured along the x axis, battery_width
        along the y axis, and battery_height along the z axis. -->
-  <xacro:property name="battery_x_offset" value="0.055"/>
+  <!-- <xacro:property name="battery_x_offset" value="0.055"/>
   <xacro:property name="battery_dist" value="0.065"/>
   <xacro:property name="battery_comp_depth" value="0.02"/>
@@ -48,5 +48,5 @@
   <xacro:property name="battery_width" value="0.047"/>
   <xacro:property name="battery_height" value="0.024"/>
-  <xacro:property name="battery_mass" value="0.5025"/>
+  <xacro:property name="battery_mass" value="0.5025"/> -->
   <!-- hub_dia and tire_dia are the diameters of the hub and tire,
        respectively. hex_hub_depth is the distance that the hex hub is
@@ -93,7 +93,7 @@
   <xacro:property name="servo_stall_torque" value="0.5649"/>
   <xacro:property name="servo_no_load_speed" value="4.553"/>
-  <material name="battery_mat">
+  <!-- <material name="battery_mat">
     <color rgba="0 0 1 1"/>
-  </material>
+  </material> -->
   <material name="chassis_mat">
     <color rgba="0.5 0.5 0.5 1"/>
@@ -142,5 +142,5 @@
   </xacro:macro>
   <!-- Battery -->
-  <xacro:macro name="battery" params="prefix reflect">
+  <!-- <xacro:macro name="battery" params="prefix reflect">
     <joint name="chassis_to_${prefix}_battery" type="fixed">
       <parent link="chassis"/>
@@ -182,5 +182,5 @@
       <material>Gazebo/Blue</material>
     </gazebo>
-  </xacro:macro>
+  </xacro:macro> -->
   <!-- Shock absorber -->
   <xacro:macro name="shock"
@@ -314,5 +314,5 @@
   </link>
   <gazebo reference="base_link">
-    <material>Gazebo/Grey</material>
+    <material>Gazebo/Blue</material>
   </gazebo>
   <!-- Chassis -->
@@ -338,5 +338,5 @@
   </link>
   <gazebo reference="chassis">
-    <material>Gazebo/Grey</material>
+    <material>Gazebo/Blue</material>
   </gazebo>
   <joint name="base_link_to_chassis" type="fixed">
@@ -345,6 +345,6 @@
   </joint>
   <!-- Batteries -->
-  <xacro:battery prefix="left" reflect="1"/>
-  <xacro:battery prefix="right" reflect="-1"/>
+  <!-- <xacro:battery prefix="left" reflect="1"/>
+  <xacro:battery prefix="right" reflect="-1"/> -->
   <!-- Wheels -->
   <xacro:front_wheel lr_prefix="left" fr_prefix="front"
@@ -359,3 +359,41 @@
     <plugin name="gazebo_ros_control" filename="libgazebo_ros_control.so"/>
   </gazebo>
+    <!-- IMU frame -->
+  <link name="imu_link">
+    <visual>
+      <geometry>
+        <box size="0.02 0.035 0.002"/>
+      </geometry>
+      <material name="Green"/>
+    </visual>
+    <inertial>
+      <mass value="0.001"/>
+      <origin xyz="0 0 0"/>
+      <inertia ixx="0.0001" ixy="0.0" ixz="0.0" iyy="0.0001" iyz="0.0" izz="0.0001"/>
+    </inertial>
+  </link>
+  <joint name="imu_joint" type="fixed">
+    <origin xyz="0 0 0" rpy="0 0 0" />
+    <parent link="base_link" />
+    <child link="imu_link" />
+  </joint>
+  <gazebo reference="imu_link">
+    <gravity>true</gravity>
+    <sensor name="imu_sensor" type="imu">
+      <always_on>true</always_on>
+      <update_rate>100</update_rate>
+      <visualize>true</visualize>
+      <plugin filename="libgazebo_ros_imu_sensor.so" name="imu_plugin">
+	      <topicName>/ackermann_vehicle/imu</topicName>
+        <bodyName>imu_link</bodyName>
+        <updateRateHZ>100.0</updateRateHZ>
+        <gaussianNoise>0.0</gaussianNoise>
+        <xyzOffset>0 0 0</xyzOffset>
+        <rpyOffset>0 0 0</rpyOffset>
+        <frameName>imu_link</frameName>
+        <initialOrientationAsReference>false</initialOrientationAsReference>
+      </plugin>
+      <pose>0 0 0 0 0 0</pose>
+    </sensor>
+  </gazebo>
 </robot>

Commit message: Changed to skateboard params

File: src/scooter_simulator/ackermann_vehicle-noetic/ackermann_vehicle_description/urdf/em_3905.urdf.xacro (robot description, xacro)
@@ -33,5 +33,5 @@
   <!-- chassis_length is measured along the x axis, chassis_width
        along the y axis, and chassis_height along the z axis. -->
-  <xacro:property name="chassis_length" value="0.258"/>
+  <xacro:property name="chassis_length" value="0.758"/>
   <xacro:property name="chassis_width" value="0.168"/>
   <xacro:property name="chassis_height" value="0.01"/>
@@ -63,5 +63,5 @@
        from a U joint to the corresponding hex hub. wheel_travel is the
        vertical wheel travel. -->
-  <xacro:property name="wheelbase" value="0.335"/>
+  <xacro:property name="wheelbase" value="0.758"/>
   <xacro:property name="hex_hub_dist" value="0.365"/>
   <xacro:property name="axle_length" value="0.03"/>
