Commit message: Added IMU link

File: src/board_model/urdf/skateboard_test.urdf (robot description, URDF)
Before this commit: robot skateboard_test, 6 links, 5 joints
Links:
- added link imu_link, mass 0.001; visual box size=0.02 0.035 0.002
Joints:
- added joint imu_joint: type fixed, parent base_link, child imu_link, origin xyz=0 0 0 rpy=0 0 0
