Commit message: Added 3D mode

File: src/board_model/urdf/skateboard_imu_Camera.urdf (robot description, URDF)
Before this commit: robot skateboard_test, 7 links, 6 joints
Links:
- added link camera_link
- added link kinect_optical_link
Joints:
- added joint camera_optical_joint: type fixed, parent base_link, child kinect_optical_link, origin xyz=0 0 0 rpy=-1.57 0 -1.57
- added joint robot_camera_joint: type fixed, parent base_link, child camera_link, origin xyz=-0.05 0.0 0.0 rpy=0.0 0.0 0.0

Commit message: Added physical model of kiect camera and coloured URDF

File: src/board_model/urdf/skateboard_imu_Camera.urdf (robot description, URDF)
Before this commit: robot skateboard_test, 9 links, 8 joints
Links:
- link camera_link: mass None -> 0.1; geometry collision box size=0.073000 0.276000 0.072000; visual mesh filename=package://board_model/models/kinect/meshes/kinect.dae
Joints:
- joint camera_optical_joint: parent base_link -> camera_link
- joint robot_camera_joint: origin xyz=-0.05 0.0 0.0 rpy=0.0 0.0 0.0 -> xyz=0.85 0.0 0.05 rpy=0.0 0.0 0.0

Commit message: Latest Board Model Changes

File: src/board_model/urdf/skateboard_imu_Camera.urdf (robot description, URDF)
Before this commit: robot skateboard_test, 9 links, 8 joints
Joints:
- joint camera_optical_joint: origin xyz=0 0 0 rpy=-1.57 0 -1.57 -> xyz=0.0 0.0 0.0 rpy=-1.57 0.0 -1.57

Commit message: Updated code for collecting data

File: src/board_model/urdf/skateboard_imu_Camera.urdf (robot description, URDF)
Before this commit: robot skateboard_test, 9 links, 8 joints
Joints:
- joint FLM: limit effort=1 velocity=1 -> effort=2 velocity=2
- joint FRM: limit effort=1 velocity=1 -> effort=2 velocity=2
- joint RLM: limit effort=1 velocity=1 -> effort=2 velocity=2
- joint RRM: limit effort=1 velocity=1 -> effort=2 velocity=2

Commit message: update perception

File: src/board_model/urdf/skateboard_imu_Camera.urdf (robot description, URDF)
Before this commit: robot mob_bot, 9 links, 8 joints
Links:
- link camera_link: mass None -> 0.1; geometry collision box size=0.073000 0.276000 0.072000; visual mesh filename=package://board_model/models/kinect/meshes/kinect.dae
Joints:
- joint FLM: limit effort=1 velocity=1 -> effort=2 velocity=2
- joint FRM: limit effort=1 velocity=1 -> effort=2 velocity=2
- joint RLM: limit effort=1 velocity=1 -> effort=2 velocity=2
- joint RRM: limit effort=1 velocity=1 -> effort=2 velocity=2
- joint camera_optical_joint: origin xyz=0 0 0 rpy=-1.57 0 -1.57 -> xyz=0.0 0.0 0.0 rpy=-1.57 0.0 -1.57; parent base_link -> camera_link
- joint robot_camera_joint: origin xyz=-0.05 0.0 0.0 rpy=0.0 0.0 0.0 -> xyz=0.85 0.0 0.05 rpy=0.0 0.0 0.0

Commit message: Final submission

File: src/board_model/urdf/skateboard_imu_Camera.urdf (robot description, URDF)
Before this commit: robot skateboard_test, 9 links, 8 joints
Links:
- link FL: mass 0.977820713429824 -> 1.77820713429824
- link FR: mass 0.977820713429824 -> 1.77820713429824
- link RL: mass 0.977820713429824 -> 1.77820713429824
- link RR: mass 0.977820713429824 -> 1.77820713429824
- link board: mass 27.3013030088211 -> 10.3013030088211
- link camera_link: mass None -> 0.1; geometry collision box size=0.073000 0.276000 0.072000; visual mesh filename=package://board_model/models/kinect/meshes/kinect.dae
Joints:
- joint FLM: limit effort=1 velocity=1 -> effort=200 velocity=200
- joint FRM: limit effort=1 velocity=1 -> effort=200 velocity=200
- joint RLM: limit effort=1 velocity=1 -> effort=200 velocity=200
- joint RRM: limit effort=1 velocity=1 -> effort=200 velocity=200
- joint camera_optical_joint: origin xyz=0 0 0 rpy=-1.57 0 -1.57 -> xyz=0.0 0.0 0.0 rpy=-1.57 0.0 -1.57; parent base_link -> camera_link
- joint robot_camera_joint: origin xyz=-0.05 0.0 0.0 rpy=0.0 0.0 0.0 -> xyz=0.85 0.0 0.05 rpy=0.0 0.0 0.0

File: src/board_model/urdf/skateboard_test.urdf (robot description, URDF)
Before this commit: robot skateboard_test, 7 links, 6 joints
Joints:
- joint FLM: limit effort=1 velocity=1 -> effort=200 velocity=100
- joint FRM: limit effort=1 velocity=1 -> effort=200 velocity=100
- joint RLM: limit effort=1 velocity=1 -> effort=200 velocity=100
- joint RRM: limit effort=1 velocity=1 -> effort=200 velocity=100
